File: Eagle/minimal_terminalv2.brd (EAGLE design)
At the start: 153.7 x 65 mm, 30 parts, among them IC1 7806T, IC2 74HC166N, X1 VGA Output

Commit message: .  updating eagle files with last fixes.
Connections:
- net RXA: now also JP2.3; no longer JP2.1
- net RXB: now also JP2.7; no longer JP2.5
- net TXA: now also JP2.1; no longer JP2.3
- net TXB: now also JP2.5; no longer JP2.7
Routing:
- net TXA: track 57.8 -> 51.8 mm
- net RXB: track 59.9 -> 56.5 mm
- net RXA: track 50.8 -> 53.4 mm
- net TXB: track 52.3 -> 54.8 mm
Changed lines of the file:
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@@
 <signal name="RXA">
 <contactref element="JP3" pad="36"/>
-<contactref element="JP2" pad="1"/>
-<wire x1="117.3861" y1="41.6052" x2="117.9576" y2="41.6052" width="0.254" layer="1"/>
-<wire x1="90.7542" y1="14.9733" x2="117.3861" y2="41.6052" width="0.254" layer="1"/>
-<wire x1="90.7542" y1="2.6289" x2="90.7542" y2="14.9733" width="0.254" layer="1"/>
-<wire x1="117.9576" y1="41.6052" x2="118.04" y2="41.68" width="0.254" layer="1"/>
-<wire x1="90.7542" y1="2.6289" x2="90.68" y2="2.6" width="0.254" layer="1"/>
-</signal>
-<signal name="TXA">
-<contactref element="JP3" pad="35"/>
 <contactref element="JP2" pad="3"/>
 <wire x1="120.4722" y1="40.005" x2="120.4722" y2="41.6052" width="0.254" layer="1"/>
@@
 <wire x1="99.3267" y1="10.8585" x2="101.9556" y2="13.4874" width="0.254" layer="1"/>
 <wire x1="96.1263" y1="10.8585" x2="99.3267" y2="10.8585" width="0.254" layer="1"/>
-<wire x1="91.7829" y1="6.5151" x2="96.1263" y2="10.8585" width="0.254" layer="1"/>
-<wire x1="91.7829" y1="2.0574" x2="91.7829" y2="6.5151" width="0.254" layer="1"/>
-<wire x1="91.2114" y1="1.4859" x2="91.7829" y2="2.0574" width="0.254" layer="1"/>
-<wire x1="89.2683" y1="1.4859" x2="91.2114" y2="1.4859" width="0.254" layer="1"/>
-<wire x1="88.2396" y1="2.5146" x2="89.2683" y2="1.4859" width="0.254" layer="1"/>
+<wire x1="90.7542" y1="5.4864" x2="96.1263" y2="10.8585" width="0.254" layer="1"/>
+<wire x1="90.7542" y1="2.6289" x2="90.7542" y2="5.4864" width="0.254" layer="1"/>
 <wire x1="120.4722" y1="41.6052" x2="120.58" y2="41.68" width="0.254" layer="1"/>
-<wire x1="88.2396" y1="2.5146" x2="88.14" y2="2.6" width="0.254" layer="1"/>
+<wire x1="90.7542" y1="2.6289" x2="90.68" y2="2.6" width="0.254" layer="1"/>
+</signal>
+<signal name="TXA">
+<contactref element="JP3" pad="35"/>
+<contactref element="JP2" pad="1"/>
+<wire x1="117.3861" y1="41.6052" x2="117.9576" y2="41.6052" width="0.254" layer="1"/>
+<wire x1="88.2396" y1="12.4587" x2="117.3861" y2="41.6052" width="0.254" layer="1"/>
+<wire x1="88.2396" y1="2.6289" x2="88.2396" y2="12.4587" width="0.254" layer="1"/>
+<wire x1="117.9576" y1="41.6052" x2="118.04" y2="41.68" width="0.254" layer="1"/>
+<wire x1="88.2396" y1="2.6289" x2="88.14" y2="2.6" width="0.254" layer="1"/>
 </signal>
 <signal name="RXB">
 <contactref element="JP4" pad="18"/>
-<contactref element="JP2" pad="5"/>
-<wire x1="124.1298" y1="41.7195" x2="123.2154" y2="41.7195" width="0.254" layer="1"/>
-<wire x1="125.1585" y1="42.7482" x2="124.1298" y2="41.7195" width="0.254" layer="1"/>
-<wire x1="129.6162" y1="42.7482" x2="125.1585" y2="42.7482" width="0.254" layer="1"/>
-<wire x1="134.3025" y1="38.0619" x2="129.6162" y2="42.7482" width="0.254" layer="1"/>
+<contactref element="JP2" pad="7"/>
+<wire x1="130.7592" y1="41.6052" x2="125.73" y2="41.6052" width="0.254" layer="1"/>
+<wire x1="134.3025" y1="38.0619" x2="130.7592" y2="41.6052" width="0.254" layer="1"/>
 <wire x1="144.2466" y1="38.0619" x2="134.3025" y2="38.0619" width="0.254" layer="1"/>
 <wire x1="146.5326" y1="35.7759" x2="144.2466" y2="38.0619" width="0.254" layer="1"/>
 <wire x1="146.5326" y1="2.6289" x2="146.5326" y2="35.7759" width="0.254" layer="1"/>
-<wire x1="123.2154" y1="41.7195" x2="123.12" y2="41.68" width="0.254" layer="1"/>
+<wire x1="125.73" y1="41.6052" x2="125.66" y2="41.68" width="0.254" layer="1"/>
 <wire x1="146.5326" y1="2.6289" x2="146.56" y2="2.6" width="0.254" layer="1"/>
 </signal>
 <signal name="TXB">
 <contactref element="JP4" pad="17"/>
-<contactref element="JP2" pad="7"/>
-<wire x1="126.5301" y1="41.6052" x2="125.73" y2="41.6052" width="0.254" layer="1"/>
-<wire x1="134.5311" y1="33.6042" x2="126.5301" y2="41.6052" width="0.254" layer="1"/>
+<contactref element="JP2" pad="5"/>
+<wire x1="124.2441" y1="41.6052" x2="123.2154" y2="41.6052" width="0.254" layer="1"/>
+<wire x1="127.7874" y1="38.0619" x2="124.2441" y2="41.6052" width="0.254" layer="1"/>
+<wire x1="130.0734" y1="38.0619" x2="127.7874" y2="38.0619" width="0.254" layer="1"/>
+<wire x1="134.5311" y1="33.6042" x2="130.0734" y2="38.0619" width="0.254" layer="1"/>
 <wire x1="134.5311" y1="32.1183" x2="134.5311" y2="33.6042" width="0.254" layer="1"/>
 <wire x1="128.3589" y1="25.9461" x2="134.5311" y2="32.1183" width="0.254" layer="1"/>
 <wire x1="128.3589" y1="18.288" x2="128.3589" y2="25.9461" width="0.254" layer="1"/>
 <wire x1="144.018" y1="2.6289" x2="128.3589" y2="18.288" width="0.254" layer="1"/>
-<wire x1="125.73" y1="41.6052" x2="125.66" y2="41.68" width="0.254" layer="1"/>
+<wire x1="123.2154" y1="41.6052" x2="123.12" y2="41.68" width="0.254" layer="1"/>
 <wire x1="144.018" y1="2.6289" x2="144.02" y2="2.6" width="0.254" layer="1"/>
 </signal>
