File: Eagle/minimal_terminalv2_rc2014.sch (EAGLE design)
At the start: 30 parts, among them IC1 7806T, IC2 74HC166N, X1 VGA Output

Commit message: .  updating eagle files with last fixes.
Connections:
- net RXA: now also JP2.3; no longer JP2.1
- net RXB: now also JP2.7; no longer JP2.5
- net TXA: now also JP2.1; no longer JP2.3
- net TXB: now also JP2.5; no longer JP2.7
Other:
- moved on the sheet: JP2, JP3, JP4, XTAL
